File: hardware/ByteSizedEncoderDecoder.kicad_sch (KiCad schematic)
At the start: 14 parts, among them J1 SM04B-SRSS-TB, J10 1x4 female header pins 0.1", J11 ICSP pads (for interfacing wi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, J2 SM04B-SRSS-TB, J3 1x4 female header pins 0.1", J4 1x4 female header pins 0.1", J5 1x4 female header pins 0.1", J6 1x4 female header pins 0.1", J7 1x4 female header pins 0.1", J8 1x4 female header pins 0.1"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

Commit message: v1.0
Other:
- company: (none) -> github.com/RCMgames/BSCD
Changed lines of the file:
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@@
 (kicad_sch (version 20230121) (generator eeschema)
   (paper "A4")
+  (title_block
+    (rev "v1.0")
+    (company "github.com/RCMgames/BSCD")
+  )
   (junction (at 118.11 81.28) (diameter 0) (color 0 0 0 0)
   )
