File: extras/hardware/ByteSizedEncoderDecoder.kicad_pcb (KiCad board)
At the start: 2 copper layers, 21.6 x 25.4 mm, 17 parts, among them J1 BM04B-SRSS-TB_LF__SN_, J10 1x4 female header pins 0.1", J11 ICSP pads, J2 BM04B-SRSS-TB_LF__SN_, J3 1x4 female header pins 0.1", J4 1x4 female header pins 0.1", J5 1x4 female header pins 0.1", J6 1x4 female header pins 0.1", J7 1x4 female header pins 0.1", J8 1x4 female header pins 0.1"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

Commit message: reorganize folder structure
Parts:
- J1, J2: value BM04B-SRSS-TB_LF__SN_ -> SM04B-SRSS-TB
- J11: value ICSP pads -> ICSP pads (for interfacing with pogo pins)
- U1: value ATMEGA328PB -> ATMEGA328PB, 32-TQFP
Changed lines of the file:
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@@
     (descr "Through hole straight pin header, 2x03, 2.54mm pitch, double rows")
     (tags "Through hole pin header THT 2x03 2.54mm double row")
-    (property "MPN" "1528-5382-ND")
+    (property "MPN" "do not purchase")
     (property "Sheetfile" "ByteSizedEncoderDecoder.kicad_sch")
     (property "Sheetname" "")
@@
         (effects (font (size 1 1) (thickness 0.15)))
     )
-    (fp_text value "ICSP pads" (at 1.27 7.41) (layer "F.Fab")
+    (fp_text value "ICSP pads (for interfacing with pogo pins)" (at 1.27 7.41) (layer "F.Fab")
         (effects (font (size 1 1) (thickness 0.15)))
     )
@@
   (footprint "parts:JST_SM04B-SRSS-TB_LF__SN_" (layer "F.Cu")
     (at 163.957 66.77 180)
-    (property "MPN" "")
-    (property "Sheetfile" "ByteSizedEncoderDecoder.kicad_sch")
-    (property "Sheetname" "")
-    (property "digikey link" "")
+    (property "MPN" "SM04B-SRSS-TB")
+    (property "Sheetfile" "ByteSizedEncoderDecoder.kicad_sch")
+    (property "Sheetname" "")
+    (property "digikey link" "455-SM04B-SRSS-TBCT-ND")
     (attr smd)
     (fp_text reference "J1" (at -4.572 4.032) (layer "F.SilkS") hide
         (effects (font (size 1.001173 1.001173) (thickness 0.15)))
     )
-    (fp_text value "BM04B-SRSS-TB_LF__SN_" (at 12.17039 5.74055) (layer "F.Fab")
+    (fp_text value "SM04B-SRSS-TB" (at 12.17039 5.74055) (layer "F.Fab")
         (effects (font (size 1.000567 1.000567) (thickness 0.15)))
     )
@@
   (footprint "parts:JST_SM04B-SRSS-TB_LF__SN_" (layer "F.Cu")
     (at 171.704 66.77 180)
-    (property "MPN" "")
-    (property "Sheetfile" "ByteSizedEncoderDecoder.kicad_sch")
-    (property "Sheetname" "")
-    (property "digikey link" "")
+    (property "MPN" "SM04B-SRSS-TB")
+    (property "Sheetfile" "ByteSizedEncoderDecoder.kicad_sch")
+    (property "Sheetname" "")
+    (property "digikey link" "455-SM04B-SRSS-TBCT-ND")
     (attr smd)
     (fp_text reference "J2" (at -0.545095 2.254) (layer "F.SilkS") hide
         (effects (font (size 1.001173 1.001173) (thickness 0.15)))
     )
-    (fp_text value "BM04B-SRSS-TB_LF__SN_" (at 12.17039 5.74055) (layer "F.Fab")
+    (fp_text value "SM04B-SRSS-TB" (at 12.17039 5.74055) (layer "F.Fab")
         (effects (font (size 1.000567 1.000567) (thickness 0.15)))
     )
@@
         (effects (font (size 1 1) (thickness 0.15)) (justify mirror))
     )
-    (fp_text value "ATMEGA328PB" (at 0 0 unlocked) (layer "B.Fab")
+    (fp_text value "ATMEGA328PB, 32-TQFP" (at 0 0 unlocked) (layer "B.Fab")
         (effects (font (size 1 1) (thickness 0.15)) (justify mirror))
     )
