File: extras/hardware/ByteSizedEncoderDecoder.kicad_sch (KiCad schematic)
At the start: 14 parts, among them J1 SM04B-SRSS-TB, J10 1x4 female header pins 0.1", J11 ICSP pads (for interfacing wi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, J2 SM04B-SRSS-TB, J3 1x4 female header pins 0.1", J4 1x4 female header pins 0.1", J5 1x4 female header pins 0.1", J6 1x4 female header pins 0.1", J7 1x4 female header pins 0.1", J8 1x4 female header pins 0.1"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

Commit message: fix link
Other:
- company: github.com/RCMgames/BSCD -> github.com/RCMgames/BSED
Changed lines of the file:
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@@
   (title_block
     (rev "v1.0")
-    (company "github.com/RCMgames/BSCD")
+    (company "github.com/RCMgames/BSED")
   )
   (junction (at 118.11 81.28) (diameter 0) (color 0 0 0 0)

Commit message: v1.1.0
Parts:
- J10, J3, J4, J5, J6, J7, J8, J9: MPN (none) -> do not place or purchase for PCB assembly; digikey link (none) -> do not place or purchase for PCB assembly
- J11: MPN do not purchase -> DNP; digikey link do not purchase -> n/a
- NT1, NT2: MPN n/a -> DNP
Changed lines of the file:
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@@
   (paper "A4")
   (title_block
-    (rev "v1.0")
+    (rev "v1.1")
     (company "github.com/RCMgames/BSED")
   )
@@
       (effects (font (size 1.27 1.27)) hide)
     )
-    (property "MPN" "" (at 27.94 101.6 0)
-      (effects (font (size 1.27 1.27)) hide)
-    )
-    (property "digikey link" "" (at 27.94 101.6 0)
+    (property "MPN" "do not place or purchase for PCB assembly" (at 27.94 101.6 0)
+      (effects (font (size 1.27 1.27)) hide)
+    )
+    (property "digikey link" "do not place or purchase for PCB assembly" (at 27.94 101.6 0)
       (effects (font (size 1.27 1.27)) hide)
     )
@@
       (effects (font (size 1.27 1.27)) hide)
     )
-    (property "MPN" "" (at 27.94 152.4 0)
-      (effects (font (size 1.27 1.27)) hide)
-    )
-    (property "digikey link" "" (at 27.94 152.4 0)
+    (property "MPN" "do not place or purchase for PCB assembly" (at 27.94 152.4 0)
+      (effects (font (size 1.27 1.27)) hide)
+    )
+    (property "digikey link" "do not place or purchase for PCB assembly" (at 27.94 152.4 0)
       (effects (font (size 1.27 1.27)) hide)
     )
@@
       (effects (font (size 1.27 1.27)) hide)
     )
-    (property "MPN" "" (at 27.94 135.89 0)
-      (effects (font (size 1.27 1.27)) hide)
-    )
-    (property "digikey link" "" (at 27.94 135.89 0)
+    (property "MPN" "do not place or purchase for PCB assembly" (at 27.94 135.89 0)
+      (effects (font (size 1.27 1.27)) hide)
+    )
+    (property "digikey link" "do not place or purchase for PCB assembly" (at 27.94 135.89 0)
       (effects (font (size 1.27 1.27)) hide)
     )
@@
       (effects (font (size 1.27 1.27)) hide)
     )
-    (property "MPN" "" (at 27.94 85.09 0)
-      (effects (font (size 1.27 1.27)) hide)
-    )
-    (property "digikey link" "" (at 27.94 85.09 0)
+    (property "MPN" "do not place or purchase for PCB assembly" (at 27.94 85.09 0)
+      (effects (font (size 1.27 1.27)) hide)
+    )
+    (property "digikey link" "do not place or purchase for PCB assembly" (at 27.94 85.09 0)
       (effects (font (size 1.27 1.27)) hide)
     )
@@
       (effects (font (size 1.27 1.27)) hide)
     )
-    (property "Datasheet" "https://www.adafruit.com/product/5382" (at 121.92 142.24 0)
-      (effects (font (size 1.27 1.27)) hide)
-    )
-    (property "MPN" "do not purchase" (at 121.92 142.24 0)
-      (effects (font (size 1.27 1.27)) hide)
-    )
-    (property "digikey link" "do not purchase" (at 121.92 142.24 0)
+    (property "Datasheet" "" (at 121.92 142.24 0)
+      (effects (font (size 1.27 1.27)) hide)
+    )
+    (property "MPN" "DNP" (at 121.92 142.24 0)
+      (effects (font (size 1.27 1.27)) hide)
+    )
+    (property "digikey link" "n/a" (at 121.92 142.24 0)
       (effects (font (size 1.27 1.27)) hide)
     )
@@
       (effects (font (size 1.27 1.27)) hide)
     )
-    (property "MPN" "n/a" (at 207.01 74.93 0)
+    (property "MPN" "DNP" (at 207.01 74.93 0)
       (effects (font (size 1.27 1.27)) hide)
     )
@@
       (effects (font (size 1.27 1.27)) hide)
     )
-    (property "MPN" "n/a" (at 207.01 77.47 0)
+    (property "MPN" "DNP" (at 207.01 77.47 0)
       (effects (font (size 1.27 1.27)) hide)
     )
@@
       (effects (font (size 1.27 1.27)) hide)
     )
-    (property "MPN" "" (at 27.94 119.38 0)
-      (effects (font (size 1.27 1.27)) hide)
-    )
-    (property "digikey link" "" (at 27.94 119.38 0)
+    (property "MPN" "do not place or purchase for PCB assembly" (at 27.94 119.38 0)
+      (effects (font (size 1.27 1.27)) hide)
+    )
+    (property "digikey link" "do not place or purchase for PCB assembly" (at 27.94 119.38 0)
       (effects (font (size 1.27 1.27)) hide)
     )
@@
       (effects (font (size 1.27 1.27)) hide)
     )
-    (property "MPN" "" (at 27.94 186.69 0)
-      (effects (font (size 1.27 1.27)) hide)
-    )
-    (property "digikey link" "" (at 27.94 186.69 0)
+    (property "MPN" "do not place or purchase for PCB assembly" (at 27.94 186.69 0)
+      (effects (font (size 1.27 1.27)) hide)
+    )
+    (property "digikey link" "do not place or purchase for PCB assembly" (at 27.94 186.69 0)
       (effects (font (size 1.27 1.27)) hide)
     )
@@
       (effects (font (size 1.27 1.27)) hide)
     )
-    (property "MPN" "" (at 27.94 168.91 0)
-      (effects (font (size 1.27 1.27)) hide)
-    )
-    (property "digikey link" "" (at 27.94 168.91 0)
+    (property "MPN" "do not place or purchase for PCB assembly" (at 27.94 168.91 0)
+      (effects (font (size 1.27 1.27)) hide)
+    )
+    (property "digikey link" "do not place or purchase for PCB assembly" (at 27.94 168.91 0)
       (effects (font (size 1.27 1.27)) hide)
     )
@@
       (effects (font (size 1.27 1.27)) hide)
     )
-    (property "MPN" "" (at 27.94 68.58 0)
-      (effects (font (size 1.27 1.27)) hide)
-    )
-    (property "digikey link" "" (at 27.94 68.58 0)
-      (effects (font (size 1.27 1.27)) hide)
-    )
+    (property "MPN" "do not place or purchase for PCB assembly" (at 27.94 68.58 0)
+      (effects (font (size 1.27 1.27)) hide)
+    )
+    (property "digikey link" "do not place or purchase for PCB assembly" (at 27.94 68.58 0)
+      (effects (font (size 1.27 1.27)) hide)
+    )
